File: 3V3-Supply.kicad_sch (KiCad schematic)
At the start: 8 parts, among them IC1 ADP2301AUJZ-R7

Commit message: updated power supply method
Parts:
- renumbered C6 to C22, C7 to C23, C8 to C24, D1 to D7
Changed lines of the file:
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@@
         )
         (path "/19e4cb9f-d0a4-4ce0-8aa4-5fe95563dc37/2757805a-b362-411e-a4a6-92c934b4db34"
-          (reference "R5") (unit 1)
+          (reference "R10") (unit 1)
         )
       )
@@
   (symbol (lib_id "HAND_PCB_V11-altium-import:GND") (at 144.78 101.6 0) (unit 1)
     (in_bom yes) (on_board yes) (dnp no)
-    (property "Reference" "#PWR015" (at 144.78 101.6 0)
+    (property "Reference" "#PWR044" (at 144.78 101.6 0)
       (effects (font (size 1.27 1.27)) hide)
     )
@@
       (project "robot-cortex"
         (path "/19e4cb9f-d0a4-4ce0-8aa4-5fe95563dc37/2757805a-b362-411e-a4a6-92c934b4db34"
-          (reference "#PWR015") (unit 1)
+          (reference "#PWR044") (unit 1)
         )
       )
@@
   (symbol (lib_id "SamacSys_Parts:NSR0530HT1G") (at 144.78 85.09 270) (unit 1)
     (in_bom yes) (on_board yes) (dnp no)
-    (property "Reference" "D1" (at 148.844 91.44 90)
+    (property "Reference" "D7" (at 148.844 91.44 90)
       (effects (font (size 1.27 1.27)) (justify left))
     )
@@
       (project "robot-cortex"
         (path "/19e4cb9f-d0a4-4ce0-8aa4-5fe95563dc37/2757805a-b362-411e-a4a6-92c934b4db34"
-          (reference "D1") (unit 1)
+          (reference "D7") (unit 1)
         )
       )
@@
   (symbol (lib_id "HAND_PCB_V11-altium-import:GND") (at 185.42 107.95 0) (unit 1)
     (in_bom yes) (on_board yes) (dnp no)
-    (property "Reference" "#PWR019" (at 185.42 107.95 0)
+    (property "Reference" "#PWR048" (at 185.42 107.95 0)
       (effects (font (size 1.27 1.27)) hide)
     )
@@
       (project "robot-cortex"
         (path "/19e4cb9f-d0a4-4ce0-8aa4-5fe95563dc37/2757805a-b362-411e-a4a6-92c934b4db34"
-          (reference "#PWR019") (unit 1)
+          (reference "#PWR048") (unit 1)
         )
       )
@@
   (symbol (lib_id "HAND_PCB_V11-altium-import:GND") (at 160.02 105.41 0) (unit 1)
     (in_bom yes) (on_board yes) (dnp no)
-    (property "Reference" "#PWR016" (at 160.02 105.41 0)
+    (property "Reference" "#PWR045" (at 160.02 105.41 0)
       (effects (font (size 1.27 1.27)) hide)
     )
@@
       (project "robot-cortex"
         (path "/19e4cb9f-d0a4-4ce0-8aa4-5fe95563dc37/2757805a-b362-411e-a4a6-92c934b4db34"
-          (reference "#PWR016") (unit 1)
+          (reference "#PWR045") (unit 1)
         )
       )
@@
   (symbol (lib_id "robot-cortex:Capacitor") (at 113.03 73.66 90) (unit 1)
     (in_bom yes) (on_board yes) (dnp no)
-    (property "Reference" "C6" (at 112.776 71.501 0)
+    (property "Reference" "C22" (at 112.776 71.501 0)
       (effects (font (size 1.27 1.27)) (justify left bottom))
     )
@@
       (project "robot-cortex"
         (path "/19e4cb9f-d0a4-4ce0-8aa4-5fe95563dc37/2757805a-b362-411e-a4a6-92c934b4db34"
-          (reference "C6") (unit 1)
+          (reference "C22") (unit 1)
         )
       )
@@
   (symbol (lib_id "robot-cortex:Capacitor") (at 168.91 87.63 0) (unit 1)
     (in_bom yes) (on_board yes) (dnp no)
-    (property "Reference" "C7" (at 170.815 88.519 0)
+    (property "Reference" "C23" (at 170.815 88.519 0)
       (effects (font (size 1.27 1.27)) (justify left bottom))
     )
@@
       (project "robot-cortex"
         (path "/19e4cb9f-d0a4-4ce0-8aa4-5fe95563dc37/2757805a-b362-411e-a4a6-92c934b4db34"
-          (reference "C7") (unit 1)
+          (reference "C23") (unit 1)
         )
       )
@@
   (symbol (lib_id "HAND_PCB_V11-altium-import:3v3") (at 172.72 81.28 180) (unit 1)
     (in_bom yes) (on_board yes) (dnp no)
-    (property "Reference" "#PWR018" (at 172.72 81.28 0)
+    (property "Reference" "#PWR046" (at 172.72 81.28 0)
       (effects (font (size 1.27 1.27)) hide)
     )
@@
       (project "robot-cortex"
         (path "/19e4cb9f-d0a4-4ce0-8aa4-5fe95563dc37/2757805a-b362-411e-a4a6-92c934b4db34"
-          (reference "#PWR018") (unit 1)
+          (reference "#PWR046") (unit 1)
         )
       )
@@
   (symbol (lib_id "HAND_PCB_V11-altium-import:GND") (at 95.25 87.63 270) (unit 1)
     (in_bom yes) (on_board yes) (dnp no)
-    (property "Reference" "#PWR03" (at 95.25 87.63 0)
+    (property "Reference" "#PWR043" (at 95.25 87.63 0)
       (effects (font (size 1.27 1.27)) hide)
     )
@@
       (project "robot-cortex"
         (path "/19e4cb9f-d0a4-4ce0-8aa4-5fe95563dc37/2757805a-b362-411e-a4a6-92c934b4db34"
-          (reference "#PWR03") (unit 1)
+          (reference "#PWR043") (unit 1)
         )
       )
@@
   (symbol (lib_id "HAND_PCB_V11-altium-import:GND") (at 172.72 95.25 0) (unit 1)
     (in_bom yes) (on_board yes) (dnp no)
-    (property "Reference" "#PWR017" (at 172.72 95.25 0)
+    (property "Reference" "#PWR047" (at 172.72 95.25 0)
       (effects (font (size 1.27 1.27)) hide)
     )
@@
       (project "robot-cortex"
         (path "/19e4cb9f-d0a4-4ce0-8aa4-5fe95563dc37/2757805a-b362-411e-a4a6-92c934b4db34"
-          (reference "#PWR017") (unit 1)
+          (reference "#PWR047") (unit 1)
         )
       )
@@
   (symbol (lib_id "robot-cortex:Capacitor") (at 176.53 87.63 0) (unit 1)
     (in_bom yes) (on_board yes) (dnp no)
-    (property "Reference" "C8" (at 178.435 88.519 0)
+    (property "Reference" "C24" (at 178.435 88.519 0)
       (effects (font (size 1.27 1.27)) (justify left bottom))
     )
@@
       (project "robot-cortex"
         (path "/19e4cb9f-d0a4-4ce0-8aa4-5fe95563dc37/2757805a-b362-411e-a4a6-92c934b4db34"
-          (reference "C8") (unit 1)
-        )
-      )
+          (reference "C24") (unit 1)
+        )
+      )
