File: ESP32.kicad_sch (KiCad schematic)
At the start: 20 parts, among them Q1 SS8050-G, Q2 SS8050-G, U7 DF52-8S-0.8H(21), U8 ESP32-WROOM-32E-H4, U9 CP2102N-A02-GQFN24R

Commit message: changed for v2
Connections:
- net NRST: now also U8.33 (IO21); no longer U8.24 (IO2)
- net at D7.2 (A), U8.6 (IO34): now also U8.8 (IO32)
Changed lines of the file:
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@@
   (junction (at 76.835 40.64) (diameter 0) (color 0 0 0 0)
+  )
+  (junction (at 87.63 73.66) (diameter 0) (color 0 0 0 0)
   )
   (junction (at 257.175 106.045) (diameter 0) (color 0 0 0 0)
@@
   (no_connect (at 211.455 128.905))
   (no_connect (at 257.175 139.065))
+  (wire (pts (xy 85.09 78.74) (xy 87.63 78.74))
+    (stroke (width 0) (type default))
+  )
   (wire (pts (xy 29.845 78.105) (xy 28.575 78.105))
     (stroke (width 0) (type default))
@@
     (stroke (width 0) (type default))
   )
+  (wire (pts (xy 87.63 78.74) (xy 87.63 73.66))
+    (stroke (width 0) (type default))
+  )
   (wire (pts (xy 29.845 70.485) (xy 28.575 70.485))
     (stroke (width 0) (type default))
@@
     (stroke (width 0) (type default))
   )
+  (wire (pts (xy 87.63 73.66) (xy 89.535 73.66))
+    (stroke (width 0) (type default))
+  )
   (wire (pts (xy 90.805 109.22) (xy 85.09 109.22))
     (stroke (width 0) (type default))
@@
     (stroke (width 0) (type default))
   )
-  (wire (pts (xy 85.09 91.44) (xy 97.155 91.44))
-    (stroke (width 0) (type default))
-  )
   (wire (pts (xy 89.535 118.11) (xy 85.09 118.11))
     (stroke (width 0) (type default))
@@
     (stroke (width 0) (type default))
   )
-  (wire (pts (xy 85.09 73.66) (xy 89.535 73.66))
+  (wire (pts (xy 88.9 111.76) (xy 85.09 111.76))
+    (stroke (width 0) (type default))
+  )
+  (wire (pts (xy 85.09 73.66) (xy 87.63 73.66))
     (stroke (width 0) (type default))
   )
@@
     (effects (font (size 1.27 1.27)) (justify left))
   )
-  (hierarchical_label "NRST" (shape input) (at 97.155 91.44 0) (fields_autoplaced)
-    (effects (font (size 1.27 1.27)) (justify left))
-  )
   (hierarchical_label "MISO" (shape input) (at 32.385 180.34 0) (fields_autoplaced)
     (effects (font (size 1.27 1.27)) (justify left))
@@
     (effects (font (size 1.27 1.27)) (justify left))
   )
+  (hierarchical_label "NRST" (shape input) (at 88.9 111.76 0) (fields_autoplaced)
+    (effects (font (size 1.27 1.27)) (justify left))
+  )

Commit message: forgto to save sch
Connections:
- net at D7.2 (A), U8.8 (IO32): no longer U8.6 (IO34)
Changed lines of the file:
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@@
   (junction (at 76.835 40.64) (diameter 0) (color 0 0 0 0)
-  )
-  (junction (at 87.63 73.66) (diameter 0) (color 0 0 0 0)
   )
   (junction (at 257.175 106.045) (diameter 0) (color 0 0 0 0)
@@
     (stroke (width 0) (type default))
   )
-  (wire (pts (xy 85.09 73.66) (xy 87.63 73.66))
-    (stroke (width 0) (type default))
-  )
