File: ESP32.kicad_sch (KiCad schematic)
At the start: 20 parts, among them Q1 SS8050-G, Q2 SS8050-G, U7 DF52-8S-0.8H(21), U8 ESP32-WROOM-32E-H4, U9 CP2102N-A02-GQFN24R

Commit message: changes that are tested+working
Connections:
- net at D7.2 (A): now also U8.8 (IO32); no longer U8.6 (IO34)
Changed lines of the file:
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@@
+    (stroke (width 0) (type default))
+  )
+  (wire (pts (xy 85.09 78.74) (xy 88.9 78.74))
     (stroke (width 0) (type default))
   )
@@
   )
   (wire (pts (xy 76.835 40.64) (xy 81.28 40.64))
+    (stroke (width 0) (type default))
+  )
+  (wire (pts (xy 88.9 78.74) (xy 88.9 73.66))
     (stroke (width 0) (type default))
   )
@@
   )
   (wire (pts (xy 48.895 76.2) (xy 49.53 76.2))
+    (stroke (width 0) (type default))
+  )
+  (wire (pts (xy 88.9 73.66) (xy 89.535 73.66))
     (stroke (width 0) (type default))
   )
@@
     (stroke (width 0) (type default))
   )
-  (wire (pts (xy 85.09 73.66) (xy 89.535 73.66))
-    (stroke (width 0) (type default))
-  )
