File: PSU_TPS63070RNMR.kicad_sch (KiCad schematic)
At the start: 9 parts, among them U10 TPS63070

Commit message: rs485
Parts:
- removed C28: C2998534, robot-cortex:C_0603_1608Metric, symbol foc-pcb:Capacitor_small
Changed lines of the file:
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@@
 (kicad_sch (version 20230121) (generator eeschema)
   (paper "A4")
-  (junction (at 171.45 78.105) (diameter 0) (color 0 0 0 0)
-  )
   (junction (at 109.22 78.105) (diameter 0) (color 0 0 0 0)
   )
@@
     (stroke (width 0) (type default))
   )
-  (wire (pts (xy 164.465 78.105) (xy 171.45 78.105))
-    (stroke (width 0) (type default))
-  )
   (wire (pts (xy 137.795 64.77) (xy 132.715 64.77))
     (stroke (width 0) (type default))
@@
     (stroke (width 0) (type default))
   )
-  (wire (pts (xy 171.45 83.185) (xy 177.8 83.185))
-    (stroke (width 0) (type default))
-  )
   (wire (pts (xy 135.89 78.105) (xy 144.145 78.105))
     (stroke (width 0) (type default))
@@
     (stroke (width 0) (type default))
   )
-  (wire (pts (xy 171.45 78.105) (xy 177.8 78.105))
+  (wire (pts (xy 164.465 78.105) (xy 177.8 78.105))
     (stroke (width 0) (type default))
   )
@@
         )
       )
-    )
-  )
-  (symbol (lib_id "foc-pcb:Capacitor_small") (at 171.45 80.645 0) (unit 1)
-    (in_bom yes) (on_board yes) (dnp no)
-    (property "Reference" "C28" (at 172.72 79.375 0)
-      (effects (font (size 1.27 1.27)) (justify left))
-    )
-    (property "Value" "C2998534" (at 171.45 76.835 90)
-      (effects (font (size 1.27 1.27)) (justify left))
-    )
-    (property "Footprint" "robot-cortex:C_0603_1608Metric" (at 172.4152 84.455 0)
-      (effects (font (size 1.27 1.27)) hide)
-    )
-    (property "Datasheet" "~" (at 171.45 80.645 0)
-      (effects (font (size 1.27 1.27)) hide)
-    )
-    (pin "1")
-    (pin "2")
-    (instances
-      (project "robot-cortex"
-        (path "/19e4cb9f-d0a4-4ce0-8aa4-5fe95563dc37/66225d13-410c-4182-8e7e-33506c71e2e4"
-          (reference "C28") (unit 1)
-        )
-        (path "/19e4cb9f-d0a4-4ce0-8aa4-5fe95563dc37/957a9604-35b3-4788-b08c-3ca047cc62dc"
-          (reference "C31") (unit 1)
-        )
-      )
-      (project "foc-pcb"
-        (path "/2b52ab19-a93e-4439-8602-a1380e4825c0"
-          (reference "C21") (unit 1)
-        )
-        (path "/2b52ab19-a93e-4439-8602-a1380e4825c0/1dc3938b-02e0-4f20-a5f4-e30fb517d809"
-          (reference "C23") (unit 1)
-        )
-      )
