File: robot-cortex.kicad_sch (KiCad schematic)
At the start: 32 parts, among them J1 USB4110GFA, M1 THRU_HOLE_PAD, M2 THRU_HOLE_PAD, U1 SPX3819M5-L-5-0, U10 DF52-4S-0.8H(21), U4 C2901617, U7 STM32G431CBT6, U8 TLE9250XSJXUMA1, U9 DF52-3S-0.8H(21)

Commit message: nearly ready to route, need to decide on 5V issue for CAN still
Parts:
- C12, C14, C16, C18, C20, C22, C24: footprint foc-pcb-library:C_0402_1005Metric -> robot-cortex:C_0402_1005Metric
- C13, C15, C17, C19, C21, C23: footprint foc-pcb-library:C_0603_1608Metric -> robot-cortex:C_0603_1608Metric
- D7: footprint foc-pcb-library:LED_0603_1608Metric -> robot-cortex:LED_0603_1608Metric
- R10: footprint foc-pcb-library:R_0402_1005Metric -> robot-cortex:R_0402_1005Metric
- U1: footprint foc-pcb-library:SOT-23-5 -> robot-cortex:SOT-23-5
- U10: footprint foc-pcb-library:DF52-4S-0.8H(21) -> robot-cortex:DF52-4S-0.8H(21)
- U4: footprint foc-pcb-library:ECS-1633-480-BN-TR -> robot-cortex:ECS-1633-480-BN-TR
- U7: footprint foc-pcb-library:LQFP48-STM32 -> robot-cortex:LQFP48-STM32
- U8: footprint foc-pcb-library:SOIC8-TLE5009 -> robot-cortex:SOIC8-TLE5009
- U9: footprint foc-pcb-library:DF52-3S-0.8H(21) -> robot-cortex:DF52-3S-0.8H(21)
Changed lines of the file:
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@@
       (effects (font (size 1.27 1.27)))
     )
-    (property "Footprint" "foc-pcb-library:DF52-4S-0.8H(21)" (at 426.085 156.845 0)
+    (property "Footprint" "robot-cortex:DF52-4S-0.8H(21)" (at 426.085 156.845 0)
       (effects (font (size 1.27 1.27)) hide)
     )
@@
       (effects (font (size 1.27 1.27)) (justify left))
     )
-    (property "Footprint" "foc-pcb-library:C_0402_1005Metric" (at 460.7052 337.82 0)
+    (property "Footprint" "robot-cortex:C_0402_1005Metric" (at 460.7052 337.82 0)
       (effects (font (size 1.27 1.27)) hide)
     )
@@
       (effects (font (size 1.27 1.27)) (justify left))
     )
-    (property "Footprint" "foc-pcb-library:C_0603_1608Metric" (at 343.2048 276.86 0)
+    (property "Footprint" "robot-cortex:C_0603_1608Metric" (at 343.2048 276.86 0)
       (effects (font (size 1.27 1.27)) hide)
     )
@@
       (effects (font (size 1.27 1.27)) (justify left))
     )
-    (property "Footprint" "foc-pcb-library:C_0603_1608Metric" (at 364.1598 276.86 0)
+    (property "Footprint" "robot-cortex:C_0603_1608Metric" (at 364.1598 276.86 0)
       (effects (font (size 1.27 1.27)) hide)
     )
@@
       (effects (font (size 1.27 1.27)))
     )
-    (property "Footprint" "foc-pcb-library:LQFP48-STM32" (at 401.955 239.395 0)
+    (property "Footprint" "robot-cortex:LQFP48-STM32" (at 401.955 239.395 0)
       (effects (font (size 1.27 1.27)) hide)
     )
@@
       (effects (font (size 1.27 1.27)) hide)
     )
-    (property "Footprint" "foc-pcb-library:R_0402_1005Metric" (at 327.025 127.635 0)
+    (property "Footprint" "robot-cortex:R_0402_1005Metric" (at 327.025 127.635 0)
       (effects (font (size 1.27 1.27)) hide)
     )
@@
       (effects (font (size 1.27 1.27)))
     )
-    (property "Footprint" "foc-pcb-library:SOIC8-TLE5009" (at 386.715 125.73 0)
+    (property "Footprint" "robot-cortex:SOIC8-TLE5009" (at 386.715 125.73 0)
       (effects (font (size 1.27 1.27)) hide)
     )
@@
       (effects (font (size 1.27 1.27)) (justify left))
     )
-    (property "Footprint" "foc-pcb-library:C_0402_1005Metric" (at 411.8102 276.86 0)
+    (property "Footprint" "robot-cortex:C_0402_1005Metric" (at 411.8102 276.86 0)
       (effects (font (size 1.27 1.27)) hide)
     )
@@
       (effects (font (size 1.27 1.27)) (justify left))
     )
-    (property "Footprint" "foc-pcb-library:C_0603_1608Metric" (at 404.7998 276.86 0)
+    (property "Footprint" "robot-cortex:C_0603_1608Metric" (at 404.7998 276.86 0)
       (effects (font (size 1.27 1.27)) hide)
     )
@@
       (effects (font (size 1.27 1.27)) (justify left))
     )
-    (property "Footprint" "foc-pcb-library:C_0603_1608Metric" (at 453.6948 337.82 0)
+    (property "Footprint" "robot-cortex:C_0603_1608Metric" (at 453.6948 337.82 0)
       (effects (font (size 1.27 1.27)) hide)
     )
@@
       (effects (font (size 1.27 1.27)))
     )
-    (property "Footprint" "foc-pcb-library:DF52-3S-0.8H(21)" (at 420.37 182.245 0)
+    (property "Footprint" "robot-cortex:DF52-3S-0.8H(21)" (at 420.37 182.245 0)
       (effects (font (size 1.27 1.27)) hide)
     )
@@
       (effects (font (size 1.27 1.27)))
     )
-    (property "Footprint" "foc-pcb-library:SOT-23-5" (at 436.245 325.12 0)
+    (property "Footprint" "robot-cortex:SOT-23-5" (at 436.245 325.12 0)
       (effects (font (size 1.27 1.27)) hide)
     )
@@
       (effects (font (size 1.27 1.27)) (justify left))
     )
-    (property "Footprint" "foc-pcb-library:C_0402_1005Metric" (at 371.1702 276.86 0)
+    (property "Footprint" "robot-cortex:C_0402_1005Metric" (at 371.1702 276.86 0)
       (effects (font (size 1.27 1.27)) hide)
     )
@@
       (effects (font (size 1.27 1.27)))
     )
-    (property "Footprint" "foc-pcb-library:ECS-1633-480-BN-TR" (at 318.135 172.085 0)
+    (property "Footprint" "robot-cortex:ECS-1633-480-BN-TR" (at 318.135 172.085 0)
       (effects (font (size 1.27 1.27)) hide)
     )
@@
       (effects (font (size 1.27 1.27)) (justify left))
     )
-    (property "Footprint" "foc-pcb-library:C_0402_1005Metric" (at 417.5252 335.915 0)
+    (property "Footprint" "robot-cortex:C_0402_1005Metric" (at 417.5252 335.915 0)
       (effects (font (size 1.27 1.27)) hide)
     )
@@
       (effects (font (size 1.27 1.27)) (justify right))
     )
-    (property "Footprint" "foc-pcb-library:LED_0603_1608Metric" (at 332.105 130.175 0)
+    (property "Footprint" "robot-cortex:LED_0603_1608Metric" (at 332.105 130.175 0)
       (effects (font (size 1.27 1.27)) hide)
     )
@@
       (effects (font (size 1.27 1.27)) (justify left))
     )
-    (property "Footprint" "foc-pcb-library:C_0402_1005Metric" (at 340.6648 180.975 0)
+    (property "Footprint" "robot-cortex:C_0402_1005Metric" (at 340.6648 180.975 0)
       (effects (font (size 1.27 1.27)) hide)
     )
@@
       (effects (font (size 1.27 1.27)) (justify left))
     )
-    (property "Footprint" "foc-pcb-library:C_0603_1608Metric" (at 410.5148 335.915 0)
+    (property "Footprint" "robot-cortex:C_0603_1608Metric" (at 410.5148 335.915 0)
       (effects (font (size 1.27 1.27)) hide)
     )
@@
       (effects (font (size 1.27 1.27)) (justify left))
     )
-    (property "Footprint" "foc-pcb-library:C_0402_1005Metric" (at 350.2152 276.86 0)
+    (property "Footprint" "robot-cortex:C_0402_1005Metric" (at 350.2152 276.86 0)
       (effects (font (size 1.27 1.27)) hide)
     )
@@
       (effects (font (size 1.27 1.27)) (justify left))
     )
-    (property "Footprint" "foc-pcb-library:C_0402_1005Metric" (at 392.1252 276.86 0)
+    (property "Footprint" "robot-cortex:C_0402_1005Metric" (at 392.1252 276.86 0)
       (effects (font (size 1.27 1.27)) hide)
     )
@@
       (effects (font (size 1.27 1.27)) (justify left))
     )
-    (property "Footprint" "foc-pcb-library:C_0603_1608Metric" (at 385.1148 276.86 0)
-      (effects (font (size 1.27 1.27)) hide)
-    )
+    (property "Footprint" "robot-cortex:C_0603_1608Metric" (at 385.1148 276.86 0)
+      (effects (font (size 1.27 1.27)) hide)
+    )

Commit message: updated power supply method
Parts:
- added R10: 470k, robot-cortex:R_0402_1005Metric, symbol foc-pcb:Resistor
- added R11: 150k, robot-cortex:R_0402_1005Metric, symbol foc-pcb:Resistor
- added R13: 680k, robot-cortex:R_0402_1005Metric, symbol foc-pcb:Resistor
- added R14: 130k, robot-cortex:R_0402_1005Metric, symbol foc-pcb:Resistor
- added R16: 0, robot-cortex:R_0402_1005Metric, symbol foc-pcb:Resistor
- U6: renamed from U1; now not fitted
- renumbered C12 to C1, C20 to C10, C21 to C11, C22 to C12, C23 to C13, C24 to C14, C13 to C2, C14 to C3, C5 to C4, C15 to C5, C16 to C6, C17 to C7, C18 to C8, C19 to C9, D6 to D1, D5 to D2, D4 to D3, D7 to D4, D1 to D5, D1 to D6, R7 to R1, R8 to R2, R10 to R3, U4 to U1, U7 to U2, U8 to U3, U9 to U4, U10 to U5
Connections:
- net +5V0: now also R16.2
- net VUSB: now also R16.1
- new net PSU_TPS63070RNMR/FB: R10.2, R11.1
- new net PSU_TPS63070RNMR/FB_GND: R11.2
- new net PSU_TPS63070RNMR/FB_VOUT: R10.1
- new net PSU_TPS63070RNMR1/FB: R13.2, R14.1
- new net PSU_TPS63070RNMR1/FB_GND: R14.2
- new net PSU_TPS63070RNMR1/FB_VOUT: R13.1
Other:
- removed sheet 3V3-Supply
- added sheet PSU_TPS63070RNMR (PSU_TPS63070RNMR.kicad_sch)
- added sheet PSU_TPS63070RNMR1 (PSU_TPS63070RNMR.kicad_sch)
- moved on the sheet: C1, C10, C11, C12, C13, C14, C2, C3, C4, C5, C6, C7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

Commit message: 3d models
Parts:
- M1, M2: footprint (none) -> robot-cortex:TEARDROP
Changed lines of the file:
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@@
       (effects (font (size 1.27 1.27)) hide)
     )
-    (property "Footprint" "" (at 147.32 125.73 0)
+    (property "Footprint" "robot-cortex:TEARDROP" (at 147.32 125.73 0)
       (effects (font (size 1.27 1.27)) hide)
     )
@@
       (effects (font (size 1.27 1.27)) hide)
     )
-    (property "Footprint" "" (at 142.24 111.76 0)
-      (effects (font (size 1.27 1.27)) hide)
-    )
+    (property "Footprint" "robot-cortex:TEARDROP" (at 142.24 111.76 0)
+      (effects (font (size 1.27 1.27)) hide)
+    )

Commit message: nothing too crazy
Parts:
- added D8: ESD9B3.3ST5G, robot-cortex:D_SOD-923, symbol robot-cortex:ESD9B3.3ST5G
Connections:
- net GND: now also D8.1 (A1)
- net VBAT: now also D8.2 (A2)

Commit message: group layouts nearly done
Parts:
- removed R2: 5.1k, robot-cortex:R_0402_1005Metric, symbol NeuralStimulatorAndRecorder:Resistor
Connections:
- net at J1.B5 (CC2): now also J1.A5 (CC1), R1.2
Changed lines of the file:
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@@
   (junction (at 206.375 147.955) (diameter 0) (color 0 0 0 0)
   )
+  (junction (at 128.27 238.125) (diameter 0) (color 0 0 0 0)
+  )
   (junction (at 203.2 163.83) (diameter 0) (color 0 0 0 0)
   )
@@
   )
   (junction (at 182.245 171.45) (diameter 0) (color 0 0 0 0)
-  )
-  (junction (at 113.03 240.665) (diameter 0) (color 0 0 0 0)
   )
   (junction (at 243.205 215.9) (diameter 0) (color 0 0 0 0)
@@
     (stroke (width 0) (type default))
   )
-  (wire (pts (xy 113.03 238.125) (xy 113.03 240.665))
+  (wire (pts (xy 113.03 238.125) (xy 113.03 243.84))
     (stroke (width 0) (type default))
   )
@@
     (stroke (width 0) (type default))
   )
-  (wire (pts (xy 113.03 243.84) (xy 113.03 240.665))
-    (stroke (width 0) (type default))
-  )
   (wire (pts (xy 157.48 106.045) (xy 160.655 106.045))
     (stroke (width 0) (type default))
@@
     (stroke (width 0) (type default))
   )
+  (wire (pts (xy 128.27 238.125) (xy 128.27 240.665))
+    (stroke (width 0) (type default))
+  )
   (wire (pts (xy 227.33 224.79) (xy 227.33 215.9))
     (stroke (width 0) (type default))
@@
     (stroke (width 0) (type default))
   )
-  (wire (pts (xy 118.11 240.665) (xy 113.03 240.665))
-    (stroke (width 0) (type default))
-  )
   (wire (pts (xy 121.285 264.795) (xy 121.285 266.065))
     (stroke (width 0) (type default))
@@
   )
   (wire (pts (xy 155.575 126.365) (xy 160.655 126.365))
-    (stroke (width 0) (type default))
-  )
-  (wire (pts (xy 125.73 240.665) (xy 128.27 240.665))
     (stroke (width 0) (type default))
   )
@@
         )
       )
-    )
-  )
-  (symbol (lib_id "NeuralStimulatorAndRecorder:Resistor") (at 121.92 240.665 90) (unit 1)
-    (in_bom yes) (on_board yes) (dnp no)
-    (property "Reference" "R2" (at 125.73 243.205 90)
-      (effects (font (size 1.27 1.27)))
-    )
-    (property "Value" "5.1k" (at 121.92 243.205 90)
-      (effects (font (size 1.27 1.27)))
-    )
-    (property "Footprint" "robot-cortex:R_0402_1005Metric" (at 109.22 245.745 0)
-      (effects (font (size 1.27 1.27)) hide)
-    )
-    (property "Datasheet" "~" (at 121.92 240.665 0)
-      (effects (font (size 1.27 1.27)) hide)
-    )
-    (pin "1")
-    (pin "2")
-    (instances
-      (project "robot-cortex"
-        (path "/19e4cb9f-d0a4-4ce0-8aa4-5fe95563dc37"
-          (reference "R2") (unit 1)
-        )
-      )
-      (project "NeuralStimulatorAndRecorder"
-        (path "/e01a8152-20cc-44b1-9878-3e8af43bcf61"
-          (reference "R1") (unit 1)
-        )
-      )

Commit message: ground planes, more routing
Parts:
- added C34: C2998534, robot-cortex:C_0603_1608Metric, symbol foc-pcb:Capacitor
- added C35: 100nF, robot-cortex:C_0402_1005Metric, symbol foc-pcb:Capacitor
Connections:
- net GND: now also C34.2, C35.2
- net VBAT: now also C34.1, C35.1
Changed lines of the file:
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@@
   (junction (at 128.27 238.125) (diameter 0) (color 0 0 0 0)
   )
+  (junction (at 191.77 201.295) (diameter 0) (color 0 0 0 0)
+  )
   (junction (at 203.2 163.83) (diameter 0) (color 0 0 0 0)
   )
@@
   )
   (junction (at 119.38 196.215) (diameter 0) (color 0 0 0 0)
+  )
+  (junction (at 191.77 208.915) (diameter 0) (color 0 0 0 0)
   )
   (junction (at 150.495 56.515) (diameter 0) (color 0 0 0 0)
@@
     (stroke (width 0) (type default))
   )
+  (wire (pts (xy 194.31 201.295) (xy 191.77 201.295))
+    (stroke (width 0) (type default))
+  )
   (wire (pts (xy 144.78 117.475) (xy 160.655 117.475))
     (stroke (width 0) (type default))
@@
     (stroke (width 0) (type default))
   )
+  (wire (pts (xy 191.77 208.915) (xy 189.23 208.915))
+    (stroke (width 0) (type default))
+  )
   (wire (pts (xy 206.375 145.415) (xy 206.375 147.955))
     (stroke (width 0) (type default))
@@
     (stroke (width 0) (type default))
   )
+  (wire (pts (xy 191.77 201.295) (xy 189.23 201.295))
+    (stroke (width 0) (type default))
+  )
   (wire (pts (xy 269.875 154.94) (xy 273.685 154.94))
     (stroke (width 0) (type default))
@@
     (stroke (width 0) (type default))
   )
+  (wire (pts (xy 194.31 208.915) (xy 191.77 208.915))
+    (stroke (width 0) (type default))
+  )
   (wire (pts (xy 163.83 264.795) (xy 163.83 262.255))
     (stroke (width 0) (type default))
@@
     (stroke (width 0) (type default))
   )
+  (wire (pts (xy 191.77 200.66) (xy 191.77 201.295))
+    (stroke (width 0) (type default))
+  )
   (wire (pts (xy 203.2 163.195) (xy 203.2 163.83))
     (stroke (width 0) (type default))
@@
   )
   (label "SS" (at 157.48 95.885 180) (fields_autoplaced)
+    (effects (font (size 1.27 1.27)) (justify right bottom))
+  )
+  (label "VBAT" (at 191.77 200.66 180) (fields_autoplaced)
     (effects (font (size 1.27 1.27)) (justify right bottom))
   )
@@
         (path "/2b52ab19-a93e-4439-8602-a1380e4825c0"
           (reference "#PWR030") (unit 1)
+        )
+      )
+    )
+  )
+  (symbol (lib_id "power:GND") (at 191.77 208.915 0) (mirror y) (unit 1)
+    (in_bom yes) (on_board yes) (dnp no) (fields_autoplaced)
+    (property "Reference" "#PWR061" (at 191.77 215.265 0)
+      (effects (font (size 1.27 1.27)) hide)
+    )
+    (property "Value" "GND" (at 191.77 213.995 0)
+      (effects (font (size 1.27 1.27)))
+    )
+    (property "Footprint" "" (at 191.77 208.915 0)
+      (effects (font (size 1.27 1.27)) hide)
+    )
+    (property "Datasheet" "" (at 191.77 208.915 0)
+      (effects (font (size 1.27 1.27)) hide)
+    )
+    (pin "1")
+    (instances
+      (project "robot-cortex"
+        (path "/19e4cb9f-d0a4-4ce0-8aa4-5fe95563dc37"
+          (reference "#PWR061") (unit 1)
+        )
+      )
+      (project "foc-pcb"
+        (path "/2b52ab19-a93e-4439-8602-a1380e4825c0"
+          (reference "#PWR032") (unit 1)
         )
       )
@@
         (path "/2b52ab19-a93e-4439-8602-a1380e4825c0"
           (reference "C9") (unit 1)
+        )
+      )
+    )
+  )
+  (symbol (lib_id "foc-pcb:Capacitor") (at 194.31 205.105 0) (unit 1)
+    (in_bom yes) (on_board yes) (dnp no)
+    (property "Reference" "C35" (at 194.945 202.565 0)
+      (effects (font (size 1.27 1.27)) (justify left))
+    )
+    (property "Value" "100nF" (at 194.945 207.645 0)
+      (effects (font (size 1.27 1.27)) (justify left))
+    )
+    (property "Footprint" "robot-cortex:C_0402_1005Metric" (at 195.2752 208.915 0)
+      (effects (font (size 1.27 1.27)) hide)
+    )
+    (property "Datasheet" "~" (at 194.31 205.105 0)
+      (effects (font (size 1.27 1.27)) hide)
+    )
+    (pin "1")
+    (pin "2")
+    (instances
+      (project "robot-cortex"
+        (path "/19e4cb9f-d0a4-4ce0-8aa4-5fe95563dc37"
+          (reference "C35") (unit 1)
+        )
+      )
+      (project "foc-pcb"
+        (path "/2b52ab19-a93e-4439-8602-a1380e4825c0"
+          (reference "C32") (unit 1)
         )
       )
@@
         )
       )
+    )
+  )
+  (symbol (lib_id "foc-pcb:Capacitor") (at 189.23 205.105 0) (mirror y) (unit 1)
+    (in_bom yes) (on_board yes) (dnp no)
+    (property "Reference" "C34" (at 188.595 203.2 0)
+      (effects (font (size 1.27 1.27)) (justify left))
+    )
+    (property "Value" "C2998534" (at 188.595 207.645 0)
+      (effects (font (size 1.27 1.27)) (justify left))
+    )
+    (property "Footprint" "robot-cortex:C_0603_1608Metric" (at 188.2648 208.915 0)
+      (effects (font (size 1.27 1.27)) hide)
+    )
+    (property "Datasheet" "~" (at 189.23 205.105 0)
+      (effects (font (size 1.27 1.27)) hide)
+    )
+    (pin "1")
+    (pin "2")
+    (instances
+      (project "robot-cortex"
+        (path "/19e4cb9f-d0a4-4ce0-8aa4-5fe95563dc37"
+          (reference "C34") (unit 1)
+        )
+      )
+      (project "foc-pcb"
+        (path "/2b52ab19-a93e-4439-8602-a1380e4825c0"
+          (reference "C5") (unit 1)
+        )
+      )

Commit message: changes that are tested+working
Parts:
- removed C1: 100nF, robot-cortex:C_0402_1005Metric, symbol foc-pcb:Capacitor
- added R2: 4.7k, robot-cortex:R_0402_1005Metric, symbol foc-pcb:Resistor
Connections:
- net GND: now also R2.2
- net NRST: now also R2.1
Changed lines of the file:
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@@
-    )
-  )
-  (symbol (lib_id "foc-pcb:Capacitor") (at 156.21 71.755 0) (mirror y) (unit 1)
-    (in_bom yes) (on_board yes) (dnp no)
-    (property "Reference" "C1" (at 155.575 69.215 0)
-      (effects (font (size 1.27 1.27)) (justify left))
-    )
-    (property "Value" "100nF" (at 155.575 74.295 0)
-      (effects (font (size 1.27 1.27)) (justify left))
-    )
-    (property "Footprint" "robot-cortex:C_0402_1005Metric" (at 155.2448 75.565 0)
-      (effects (font (size 1.27 1.27)) hide)
-    )
-    (property "Datasheet" "~" (at 156.21 71.755 0)
-      (effects (font (size 1.27 1.27)) hide)
-    )
-    (pin "1")
-    (pin "2")
-    (instances
-      (project "robot-cortex"
-        (path "/19e4cb9f-d0a4-4ce0-8aa4-5fe95563dc37"
-          (reference "C1") (unit 1)
-        )
-      )
-      (project "foc-pcb"
-        (path "/2b52ab19-a93e-4439-8602-a1380e4825c0"
-          (reference "C3") (unit 1)
-        )
-      )
     )
   )
@@
         )
       )
+    )
+  )
+  (symbol (lib_id "foc-pcb:Resistor") (at 156.21 71.755 0) (mirror y) (unit 1)
+    (in_bom yes) (on_board yes) (dnp no)
+    (property "Reference" "R2" (at 154.94 72.39 0)
+      (effects (font (size 1.27 1.27)) (justify left))
+    )
+    (property "Value" "4.7k" (at 152.4 74.295 0)
+      (effects (font (size 1.27 1.27)))
+    )
+    (property "Footprint" "robot-cortex:R_0402_1005Metric" (at 161.29 59.055 0)
+      (effects (font (size 1.27 1.27)) hide)
+    )
+    (property "Datasheet" "~" (at 156.21 71.755 0)
+      (effects (font (size 1.27 1.27)) hide)
+    )
+    (pin "1")
+    (pin "2")
+    (instances
+      (project "robot-cortex"
+        (path "/19e4cb9f-d0a4-4ce0-8aa4-5fe95563dc37"
+          (reference "R2") (unit 1)
+        )
+      )

Commit message: rs485
Parts:
- added C1, C36: 100nF, Capacitor_SMD:C_0402_1005Metric, symbol Device:C
- added IC1: THVD2410VDRCR, robot-cortex:THVD2410VDRCR, symbol SamacSys_Parts:THVD2410VDRCR
- added R18, R20: 1k, robot-cortex:R_0402_1005Metric, symbol robot-cortex:R
- added R19: 120, robot-cortex:R_0402_1005Metric, symbol robot-cortex:R
Connections:
- net +3V3: now also C1.2, IC1.1 (VIO)
- net +5V0: now also C36.2, IC1.10 (VCC), R18.2
- net GND: now also C1.1, C36.1, IC1.11 (EP_1), IC1.12 (EP_2), IC1.13 (EP_3), IC1.14 (EP_4), IC1.15 (EP_5), IC1.6 (GND), IC1.7 (SLR), R20.1
- net UART1_RX: now also IC1.2 (R)
- net UART1_TX: now also IC1.5 (D)
- net UART1_DE: now reaches U2.30 (PA8)
- net UART1_DE: now also IC1.3 (DE), IC1.4 (~{RE})
- net CANH renamed A-PROTECTED
- net A-PROTECTED: now also IC1.8 (A), R19.1, R20.2
- net CANL renamed B-PROTECTED
- net B-PROTECTED: now also IC1.9 (B), R18.1, R19.2
Other:
- moved on the sheet: U5
